File: blinky.kicad_sch (KiCad schematic)
At the start: 7 parts, among them U1 7555

Commit message: Layout board
Other:
- title: (none) -> Getting to Blinky
Changed lines of the file:
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@@
 	(generator_version "8.0")
 	(paper "A5")
+	(title_block
+		(title "Getting to Blinky")
+		(date "2025-06-22")
+		(rev "0.1")
+	)
 	(junction
 		(at 91.44 53.34)

Commit message: Add fabrication files
Parts:
- C1: value 1U -> 1uf
Changed lines of the file:
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@@
 			)
 		)
-		(property "Value" "1U"
+		(property "Value" "1uf"
 			(at 95.25 69.8499 0)
 			(effects
